Commit message: Replace EC616 end-effector viz with KWR75 + AG95 meshes.
Mount the force/torque sensor between Link6 flange and the AG95 gripper in the Three.js URDF, and cache-bust the model URL so browsers pick up the new assets.

Co-authored-by: Cursor <cursoragent@cursor.com>

File: src/sensors_dcs/static/models/ec616/ec616.urdf (robot description, URDF)
Before this commit: robot ec616, 10 links, 9 joints
Links:
- removed link gripper_1_link
- removed link gripper_2_link
- added link ft_kwr75_link, mass 0.25; collision mesh filename=meshes/KWR75.STL; visual mesh filename=meshes/KWR75.STL
- link gripper_centor_link: mass 0.05 -> 0.8; geometry collision mesh filename=meshes/AG95.STL; visual mesh filename=meshes/AG95.STL
Joints:
- removed joint gripper_1_joint
- removed joint gripper_2_joint
- added joint ft_kwr75_fixed: type fixed, parent Link6, child ft_kwr75_link, origin xyz=0 0 0 rpy=0 0 0
- joint gripper_centor_fixed: origin xyz=0 0 0.025 rpy=0 0 0 -> xyz=0 0 0.0335 rpy=0 0 0; parent Link6 -> ft_kwr75_link
